Commit message: 0928Test

File: src/arm_planning/arm_kinematics_solver/models/AUBO_HRM.urdf (robot description, URDF)
Before this commit: robot AUBO_HRM, 19 links, 18 joints
Links:
- link left_link0: mass 1.036000 -> 1.065000
- link left_link1: mass 0.222000 -> 0.254000
- link left_link2: mass 1.226000 -> 1.258000
- link left_link3: mass 1.824000 -> 1.810000
- link left_link4: mass 0.123000 -> 0.155000
- link left_link5: mass 1.010000 -> 1.191000
- link left_link6: mass 0.487000 -> 0.519000
- link left_link7: mass 0.228000 -> 0.212000
- link right_link0: mass 1.036000 -> 1.065000
- link right_link1: mass 0.222000 -> 0.254000
- link right_link2: mass 1.226000 -> 1.258000
- link right_link3: mass 1.824000 -> 1.810000
- link right_link4: mass 0.123000 -> 0.155000
- link right_link5: mass 1.010000 -> 1.191000
- link right_link6: mass 0.487000 -> 0.519000
- link right_link7: mass 0.228000 -> 0.212000
Joints:
- joint left_flange: origin xyz=0 -0.1115 0 rpy=1.5707963267948966192313216916398 0 0 -> xyz=0 -0.084 0 rpy=1.5707963267948966192313216916398 0 0
- joint left_joint1: limit lower=-3.14159265358979 upper=0.785398163397448 effort=40 velocity=3.14159265358979 -> lower=-3.14159265358979 upper=1.785398163397448 effort=40 velocity=3.14159265358979
- joint left_joint4: limit lower=-2.26892802759263 upper=0 effort=22 velocity=4.18879020478639 -> lower=0 upper=2.26892802759263 effort=22 velocity=4.18879020478639
- joint right_flange: origin xyz=0 -0.1115 0 rpy=1.5707963267948966192313216916398 0 0 -> xyz=0 -0.084 0 rpy=1.5707963267948966192313216916398 0 0
- joint right_joint1: limit lower=-0.785398163397448 upper=3.14159265358979 effort=40 velocity=3.14159265358979 -> lower=-1.785398163397448 upper=3.14159265358979 effort=40 velocity=3.14159265358979
- joint right_joint2: limit lower=-1.74532925199433 upper=0 effort=40 velocity=3.14159265358979 -> lower=-1.74532925199433 upper=0.17 effort=40 velocity=3.14159265358979
- joint right_joint4: limit lower=0 upper=2.26892802759263 effort=22 velocity=4.18879020478639 -> lower=-2.26892802759263 upper=0 effort=22 velocity=4.18879020478639
- joint right_joint5: limit lower=-2.26892802759263 upper=2.26892802759263 effort=8 velocity=3.14159265358979 -> lower=-3.14 upper=3.14 effort=8 velocity=3.14159265358979

File: src/arm_planning/aubo_arm_urdf/aubo_arm_l/urdf/AUBO_HRM_L.urdf (robot description, URDF)
Before this commit: robot aubo_arm_l, 10 links, 9 joints
Links:
- link link0: mass 1.036000 -> 1.065000; geometry collision mesh filename=package://aubo_description/meshes/AUBO_HRA_L/collision/link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; visual mesh filename=package://aubo_description/meshes/AUBO_HRA_L/visual/link0.S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
- link link1: mass 0.222000 -> 0.254000; geometry collision mesh filename=package://aubo_description/meshes/AUBO_HRA_L/collision/link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; visual mesh filename=package://aubo_description/meshes/AUBO_HRA_L/visual/link1.S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
- link link2: mass 1.226000 -> 1.258000; geometry collision mesh filename=package://aubo_description/meshes/AUBO_HRA_L/collision/link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; visual mesh filename=package://aubo_description/meshes/AUBO_HRA_L/visual/link2.S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
- link link3: mass 1.824000 -> 1.810000; geometry collision mesh filename=package://aubo_description/meshes/AUBO_HRA_L/collision/link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; visual mesh filename=package://aubo_description/meshes/AUBO_HRA_L/visual/link3.S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
- link link4: mass 0.123000 -> 0.155000; geometry collision mesh filename=package://aubo_description/meshes/AUBO_HRA_L/collision/link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; visual mesh filename=package://aubo_description/meshes/AUBO_HRA_L/visual/link4.S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
- link link5: mass 1.010000 -> 1.191000; geometry collision mesh filename=package://aubo_description/meshes/AUBO_HRA_L/collision/link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; visual mesh filename=package://aubo_description/meshes/AUBO_HRA_L/visual/link5.S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
- link link6: mass 0.487000 -> 0.519000; geometry collision mesh filename=package://aubo_description/meshes/AUBO_HRA_L/collision/link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; visual mesh filename=package://aubo_description/meshes/AUBO_HRA_L/visual/link6.S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
- link link7: mass 0.228000 -> 0.212000; geometry collision mesh filename=package://aubo_description/meshes/AUBO_HRA_L/collision/link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; visual mesh filename=package://aubo_description/meshes/AUBO_HRA_L/visual/link7.S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
Joints:
- joint flange: origin xyz=0 -0.1115 0 rpy=1.5707963267948966192313216916398 0 0 -> xyz=0 -0.084 0 rpy=1.5707963267948966192313216916398 0 0

File: src/arm_planning/aubo_arm_urdf/aubo_arm_r/urdf/AUBO_HRM_R.urdf (robot description, URDF)
Before this commit: robot aubo_arm_r, 10 links, 9 joints
Links:
- link link0: mass 1.036000 -> 1.065000; geometry collision mesh filename=package://aubo_description/meshes/AUBO_HRA_R/collision/link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; visual mesh filename=package://aubo_description/meshes/AUBO_HRA_R/visual/link0.S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
- link link1: mass 0.222000 -> 0.254000; geometry collision mesh filename=package://aubo_description/meshes/AUBO_HRA_R/collision/link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; visual mesh filename=package://aubo_description/meshes/AUBO_HRA_R/visual/link1.S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
- link link2: mass 1.226000 -> 1.258000; geometry collision mesh filename=package://aubo_description/meshes/AUBO_HRA_R/collision/link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; visual mesh filename=package://aubo_description/meshes/AUBO_HRA_R/visual/link2.S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
- link link3: mass 1.824000 -> 1.810000; geometry collision mesh filename=package://aubo_description/meshes/AUBO_HRA_R/collision/link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; visual mesh filename=package://aubo_description/meshes/AUBO_HRA_R/visual/link3.S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
- link link4: mass 0.123000 -> 0.155000; geometry collision mesh filename=package://aubo_description/meshes/AUBO_HRA_R/collision/link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; visual mesh filename=package://aubo_description/meshes/AUBO_HRA_R/visual/link4.S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
- link link5: mass 1.010000 -> 1.191000; geometry collision mesh filename=package://aubo_description/meshes/AUBO_HRA_R/collision/link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; visual mesh filename=package://aubo_description/meshes/AUBO_HRA_R/visual/link5.S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
- link link6: mass 0.487000 -> 0.519000; geometry collision mesh filename=package://aubo_description/meshes/AUBO_HRA_R/collision/link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; visual mesh filename=package://aubo_description/meshes/AUBO_HRA_R/visual/link6.S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
- link link7: mass 0.228000 -> 0.212000; geometry collision mesh filename=package://aubo_description/meshes/AUBO_HRA_R/collision/link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; visual mesh filename=package://aubo_description/meshes/AUBO_HRA_R/visual/link7.S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
Joints:
- joint flange: origin xyz=0 -0.1115 0 rpy=1.5707963267948966192313216916398 0 0 -> xyz=0 -0.084 0 rpy=1.5707963267948966192313216916398 0 0
