Commit message: 添加rviz

File: src/arm_planning/test_planning/model/humanoid.urdf (robot description, URDF)
Before this commit: robot humanoid, 57 links, 56 joints
Links:
- link pelvis: geometry visual mesh filename=package://test_planning/meshes/pelvis.STL
Joints:
- joint waist_yaw_joint: limit (none) -> lower=-2.96 upper=2.96 effort=90 velocity=15

Commit message: 开放基座yaw 以左臂为主进行了运动学优化，更改零空间阻抗目标位置

File: src/arm_planning/test_planning/model/humanoid.urdf (robot description, URDF)
Before this commit: robot humanoid, 57 links, 56 joints
Joints:
- joint waist_yaw_joint: limit lower=-2.96 upper=2.96 effort=90 velocity=15 -> lower=-1 upper=1 effort=90 velocity=15; type fixed -> revolute

Commit message: HQP

File: src/arm_planning/test_planning/model/humanoid.urdf (robot description, URDF)
Before this commit: robot humanoid, 57 links, 56 joints
Links:
- added link waist_Z_link, mass 1; visual cylinder length=0.1 radius=0.05
- added link waist_pitch_link, mass 0.0001; visual cylinder length=0.1 radius=0.05
- added link waist_roll_link, mass 0.0001; visual cylinder length=0.1 radius=0.05
Joints:
- added joint waist_Z_joint: type prismatic, parent pelvis, child waist_Z_link, origin xyz=0 0 -0.0755 rpy=0 0 0, axis 0 0 1, limit lower=-0.15 upper=0 effort=90 velocity=0.5
- added joint waist_pitch_joint: type revolute, parent waist_roll_link, child waist_pitch_link, origin xyz=0 0 0 rpy=0 0 0, axis 0 1 0, limit lower=-0.25 upper=0.25 effort=90 velocity=0.4
- added joint waist_roll_joint: type revolute, parent waist_Z_link, child waist_roll_link, origin xyz=0 0 0 rpy=0 0 0, axis 1 0 0, limit lower=-0.25 upper=0.25 effort=90 velocity=0.4
- joint waist_yaw_joint: origin xyz=0 0 -0.0755 rpy=0 0 0 -> xyz=0 0 0 rpy=0 0 0; parent pelvis -> waist_pitch_link

Commit message: 2025

File: src/arm_planning/test_planning/model/humanoid.urdf (robot description, URDF)
Before this commit: robot humanoid, 60 links, 59 joints
Links:
- link L_hand_base_link: geometry visual mesh filename=package://test_planning/model2/meshes/L_hand_base_link.STL
- link L_index_intermediate: geometry visual mesh filename=package://test_planning/model2/meshes/Link16_L.STL
- link L_index_proximal: geometry visual mesh filename=package://test_planning/model2/meshes/Link15_L.STL
- link L_middle_intermediate: geometry visual mesh filename=package://test_planning/model2/meshes/Link18_L.STL
- link L_middle_proximal: geometry visual mesh filename=package://test_planning/model2/meshes/Link17_L.STL
- link L_pinky_intermediate: geometry visual mesh filename=package://test_planning/model2/meshes/Link22_L.STL
- link L_pinky_proximal: geometry visual mesh filename=package://test_planning/model2/meshes/Link21_L.STL
- link L_ring_intermediate: geometry visual mesh filename=package://test_planning/model2/meshes/Link20_L.STL
- link L_ring_proximal: geometry visual mesh filename=package://test_planning/model2/meshes/Link19_L.STL
- link L_thumb_distal: geometry visual mesh filename=package://test_planning/model2/meshes/Link14_L.STL
- link L_thumb_intermediate: geometry visual mesh filename=package://test_planning/model2/meshes/Link13_L.STL
- link L_thumb_proximal: geometry visual mesh filename=package://test_planning/model2/meshes/Link12_L.STL
- link L_thumb_proximal_base: geometry visual mesh filename=package://test_planning/model2/meshes/Link11_L.STL
- link R_hand_base_link: geometry visual mesh filename=package://test_planning/model2/meshes/R_hand_base_link.STL
- link R_index_intermediate: geometry visual mesh filename=package://test_planning/model2/meshes/Link16_R.STL
- link R_index_proximal: geometry visual mesh filename=package://test_planning/model2/meshes/Link15_R.STL
- link R_middle_intermediate: geometry visual mesh filename=package://test_planning/model2/meshes/Link18_R.STL
- link R_middle_proximal: geometry visual mesh filename=package://test_planning/model2/meshes/Link17_R.STL
- link R_pinky_intermediate: geometry visual mesh filename=package://test_planning/model2/meshes/Link22_R.STL
- link R_pinky_proximal: geometry visual mesh filename=package://test_planning/model2/meshes/Link21_R.STL
- link R_ring_intermediate: geometry visual mesh filename=package://test_planning/model2/meshes/Link20_R.STL
- link R_ring_proximal: geometry visual mesh filename=package://test_planning/model2/meshes/Link19_R.STL
- link R_thumb_distal: geometry visual mesh filename=package://test_planning/model2/meshes/Link14_R.STL
- link R_thumb_intermediate: geometry visual mesh filename=package://test_planning/model2/meshes/Link13_R.STL
- link R_thumb_proximal: geometry visual mesh filename=package://test_planning/model2/meshes/Link12_R.STL
- link R_thumb_proximal_base: geometry visual mesh filename=package://test_planning/model2/meshes/Link11_R.STL
- link arm_base_l_link: geometry visual mesh filename=package://test_planning/model2/meshes/arm_base_l_link.STL
- link arm_base_r_link: geometry visual mesh filename=package://test_planning/model2/meshes/arm_base_r_link.STL
- link arm_yaw_l_link: geometry visual mesh filename=package://test_planning/model2/meshes/arm_yaw_l_link.STL
- link arm_yaw_r_link: geometry visual mesh filename=package://test_planning/model2/meshes/arm_yaw_r_link.STL
- link elbow_pitch_l_link: geometry collision sphere radius=0.035; visual mesh filename=package://test_planning/model2/meshes/elbow_pitch_l_link.STL
- link elbow_pitch_r_link: geometry collision sphere radius=0.035; visual mesh filename=package://test_planning/model2/meshes/elbow_pitch_r_link.STL
- link elbow_yaw_l_link: geometry collision mesh filename=package://test_planning/model2/meshes/elbow_yaw_l_link.STL; visual mesh filename=package://test_planning/model2/meshes/elbow_yaw_l_link.STL
- link elbow_yaw_r_link: geometry visual mesh filename=package://test_planning/model2/meshes/elbow_yaw_r_link.STL
- link head_base_link: geometry visual mesh filename=package://test_planning/model2/meshes/head_base_link.STL
- link head_yaw_link: geometry visual mesh filename=package://test_planning/model2/meshes/head_yaw_link.STL
- link pelvis: geometry visual mesh filename=package://test_planning/model2/meshes/pelvis.STL
- link shoulder_pitch_l_link: geometry visual mesh filename=package://test_planning/model2/meshes/shoulder_pitch_l_link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
- link shoulder_pitch_r_link: geometry visual mesh filename=package://test_planning/model2/meshes/shoulder_pitch_r_link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
- link shoulder_roll_l_link: geometry collision sphere radius=0.035; visual mesh filename=package://test_planning/model2/meshes/shoulder_roll_l_link.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
- link shoulder_roll_r_link: geometry collision sphere radius=0.035; visual mesh filename=package://test_planning/model2/meshes/shoulder_roll_r_link.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
- link waist_link: geometry visual cylinder length=0.3 radius=0.08; visual mesh filename=package://test_planning/model2/meshes/waist_link1.stl
- link wrist_pitch_l_link: geometry visual mesh filename=package://test_planning/model2/meshes/wrist_pitch_l_link.STL
- link wrist_pitch_r_link: geometry visual mesh filename=package://test_planning/model2/meshes/wrist_pitch_r_link.STL
- link wrist_roll_l_link: geometry visual mesh filename=package://test_planning/model2/meshes/wrist_roll_l_link.STL
- link wrist_roll_r_link: geometry visual mesh filename=package://test_planning/model2/meshes/wrist_roll_r_link.STL
Joints:
- joint waist_pitch_joint: type revolute -> fixed
