Commit message: 至此max运动学开发完毕

File: src/arm_planning/test_planning/model2/urdf/dual_arm_description.urdf (robot description, URDF)
Before this commit: robot dual_arm_description, 24 links, 23 joints
Joints:
- joint pelvis_joint: origin xyz=0.0 0 -0.00599999999999996 rpy=0 0 0 -> xyz=0.0 0 -0.006 rpy=0 0 0

File: src/arm_planning/test_planning/x_humanoid_ultra_noeyes/urdf/humanoid.urdf (robot description, URDF)
Before this commit: robot humanoid, 26 links, 25 joints
Links:
- added link base_footprint
- link pelvis: mass 4.585  -> None
Joints:
- added joint base_link_joint: type fixed, parent base_footprint, child pelvis, origin xyz=0 0 1.08 rpy=0 0 0, axis 0 0 0
